Commit message: Update puppy.urdf

File: puppy/urdf/puppy.urdf (robot description, URDF)
Before this commit: robot puppy, 14 links, 13 joints
Links:
- link BLendeffoctor: geometry collision mesh filename=package://puppy2/meshes/BLendeffoctor.STL; visual mesh filename=package://puppy2/meshes/BLendeffoctor.STL
- link BLlower: geometry collision mesh filename=package://puppy2/meshes/BLlower.STL; visual mesh filename=package://puppy2/meshes/BLlower.STL
- link BLupper: geometry collision mesh filename=package://puppy2/meshes/BLupper.STL; visual mesh filename=package://puppy2/meshes/BLupper.STL
- link BRendeffector: geometry collision mesh filename=package://puppy2/meshes/BRendeffector.STL; visual mesh filename=package://puppy2/meshes/BRendeffector.STL
- link BRlower: geometry collision mesh filename=package://puppy2/meshes/BRlower.STL; visual mesh filename=package://puppy2/meshes/BRlower.STL
- link BRupper: geometry collision mesh filename=package://puppy2/meshes/BRupper.STL; visual mesh filename=package://puppy2/meshes/BRupper.STL
- link FLendeffector: geometry collision mesh filename=package://puppy2/meshes/FLendeffector.STL; visual mesh filename=package://puppy2/meshes/FLendeffector.STL
- link FLlower: geometry collision mesh filename=package://puppy2/meshes/FLlower.STL; visual mesh filename=package://puppy2/meshes/FLlower.STL
- link FLupper: geometry collision mesh filename=package://puppy2/meshes/FLupper.STL; visual mesh filename=package://puppy2/meshes/FLupper.STL
- link FRendeffector: geometry collision mesh filename=package://puppy2/meshes/FRendeffector.STL; visual mesh filename=package://puppy2/meshes/FRendeffector.STL
- link FRlower: geometry collision mesh filename=package://puppy2/meshes/FRlower.STL; visual mesh filename=package://puppy2/meshes/FRlower.STL
- link FRupper: geometry collision mesh filename=package://puppy2/meshes/FRupper.STL; visual mesh filename=package://puppy2/meshes/FRupper.STL
- link base: geometry collision mesh filename=package://puppy2/meshes/base.STL; visual mesh filename=package://puppy2/meshes/base.STL
- link spine: geometry collision mesh filename=package://puppy2/meshes/spine.STL; visual mesh filename=package://puppy2/meshes/spine.STL
